File: arduino-hat/mega_shield.kicad_pcb (KiCad board)
At the start: 2 copper layers, 101.6 x 53.3 mm, 72 parts, among them IC1 1870_LD1117S50CTR, IC3 ATMEGA2560-15AU, IC4 ATMEGA16U2-MU, IC6 LP2985-33DBVR, IC7 LMV358IDGKR, T1 PMV48XP, X1 POWERSUPPLY_DC21MMX, Y1 CSTCE16M0V53-R0, Y2 16MHz

Commit message: Update mega_shield.kicad_pcb
Parts:
- removed C1, C14, C15: 22p, MEGA2560_Rev3e:C0603-ROUND
- removed C10, C13: 1uF, MEGA2560_Rev3e:C0603-ROUND
- removed C11, C12, C16, C2, C3, C4, C5, C6, C7, C8, C9: 100nF, MEGA2560_Rev3e:C0603-ROUND
- removed D1: M7, MEGA2560_Rev3e:SMB
- removed D2, D3: CD1206-S01575, MEGA2560_Rev3e:MINIMELF
- removed F1: MF-MSMF050-2 500mA, MEGA2560_Rev3e:L1812
- removed FD1, FD2, FD3, FD4: FIDUCIALMOUNT, MEGA2560_Rev3e:FIDUCIA-MOUNT
- removed GROUND0, RESET-EN0: , MEGA2560_Rev3e:SJ
- removed IC1: 1870_LD1117S50CTR, MEGA2560_Rev3e:LINEAR_SOT223
- removed IC3: ATMEGA2560-15AU, MEGA2560_Rev3e:TQFP100
- removed IC4: ATMEGA16U2-MU, MEGA2560_Rev3e:MLF32
- removed IC6: LP2985-33DBVR, MEGA2560_Rev3e:SOT23-DBV
- removed IC7: LMV358IDGKR, MEGA2560_Rev3e:MSOP08
- removed ICSP0: ICSP, MEGA2560_Rev3e:2X03
- removed L0, RX0, TX0: Yellow, MEGA2560_Rev3e:CHIPLED_0805
- removed L1: MH2029-300Y, MEGA2560_Rev3e:0805
- removed L2: 10uH, MEGA2560_Rev3e:0805
- removed ON0: Green, MEGA2560_Rev3e:CHIPLED_0805
- removed PC1, PC2: 47uF, MEGA2560_Rev3e:PANASONIC_D
- removed R1, R2: 1M, MEGA2560_Rev3e:R0603-ROUND
- removed RESET0: TS42, MEGA2560_Rev3e:TS42
- removed RN1, RN5: 10k, MEGA2560_Rev3e:CAY16
- removed RN2: 22R, MEGA2560_Rev3e:CAY16
- removed RN3, RN4: 1K, MEGA2560_Rev3e:CAY16
- removed T1: PMV48XP, MEGA2560_Rev3e:SOT-23
- removed UNK_HOLE_3: , MEGA2560_Rev3e:dummyfp3
- removed UNK_HOLE_4: , MEGA2560_Rev3e:dummyfp4
- removed UNK_HOLE_5: , MEGA2560_Rev3e:dummyfp5
- removed X1: POWERSUPPLY_DC21MMX, MEGA2560_Rev3e:POWERSUPPLY_DC-21MM
- removed X2: , MEGA2560_Rev3e:PN61729
- removed Y1: CSTCE16M0V53-R0, MEGA2560_Rev3e:RESONATOR
- removed Y2: 16MHz, MEGA2560_Rev3e:QS
- removed Z1, Z2: BRNCG0603MLC-05E, MEGA2560_Rev3e:CT_CN0603
Routing:
- net +5V: track 345.7 -> 0.18 mm, vias 24 -> 0
- net RESET: track 202.0 -> 0.00 mm, vias 5 -> 0
- net SCL: track 167.5 -> 0.51 mm, vias 4 -> 0
- net SDA: track 159.0 -> 0.13 mm, vias 4 -> 0
- net PB3: track 115.4 -> 7.33 mm, vias 3 -> 0
- net PB2: track 104.5 -> 0.00 mm, vias 3 -> 0
- net PB1: track 91.3 -> 0.00 mm, vias 3 -> 0
- net ADC13: track 75.7 -> 0.00 mm, vias 1 -> 0
- net ADC14: track 73.4 -> 0.00 mm, vias 1 -> 0
- net N$3: track 71.9 -> 0.00 mm, vias 4 -> 0
- net ADC11: track 71.6 -> 0.00 mm, vias 1 -> 0
- net ADC12: track 71.5 -> 0.00 mm, vias 1 -> 0
- net ADC15: track 71.3 -> 0.00 mm, vias 1 -> 0
- net PB0: track 66.4 -> 0.00 mm, vias 2 -> 0
- net ADC10: track 65.2 -> 0.00 mm, vias 1 -> 0
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- removed copper zone on B.Cu, net +5V
- removed copper zone on F.Cu, net +5V
Other:
- board text removed: "28"
- board text removed: "30"
- board text removed: "32"
- board text removed: "34"
- board text removed: "36"
- board text removed: "38"
- board text removed: "3V3"
- board text removed: "40"
- board text removed: "42"
- board text removed: "44"
- board text removed: "46"
- board text removed: "48"
- board text removed: "50"
- board text removed: "52"
- board text removed: "ANALOG IN"
- board text removed: "Arduino"
- board text removed: "Arduino.org"
- board text removed: "DIGITAL"
- board text removed: "IOREF"
- board text removed: "ITALY"
- board text removed: "L"
- board text removed: "MADE IN"
- board text removed: "MEGA 2560"
- board text removed: "ON"
- board text removed: "PC1"
- board text removed: "PC2"
- board text removed: "RESET"
- board text removed: "TM"
- board text removed: "VIN"
- board text removed: "designed by"
- board text removed: "tinker it"
