File: arduino-hat/arduino-hat.kicad_pcb (KiCad board)
At the start: 2 copper layers, 0 parts

Commit message: more PCB work
Parts:
- added A1: Arduino_Mega2560_R3_Shield, PCM_arduino-library:Arduino_Mega2560_R3_Shield, F.Cu at (93.4, 120.4)
- added C1: 0.01F, Capacitor_SMD:C_1210_3225Metric_Pad1.33x2.70mm_HandSolder, F.Cu at (138.5, 104.6)
- added C2: 0.01F, Capacitor_SMD:C_1210_3225Metric_Pad1.33x2.70mm_HandSolder, F.Cu at (121.5, 110.1)
- added C3: 10 uF, Capacitor_SMD:C_1210_3225Metric_Pad1.33x2.70mm_HandSolder, F.Cu at (121.5, 78.9)
- added C4: 0.01, Capacitor_SMD:C_1210_3225Metric_Pad1.33x2.70mm_HandSolder, F.Cu at (138.5, 97.5)
- added C5: 0.01, Capacitor_SMD:C_1210_3225Metric_Pad1.33x2.70mm_HandSolder, F.Cu at (158.5, 75.3)
- added C8: 0.01, Capacitor_SMD:C_1210_3225Metric_Pad1.33x2.70mm_HandSolder, F.Cu at (138.5, 90.6)
- added C9: 0.01, Capacitor_SMD:C_1210_3225Metric_Pad1.33x2.70mm_HandSolder, F.Cu at (127.9, 89.5)
- added D1: LED, LED_SMD:LED_1210_3225Metric_Pad1.42x2.65mm_HandSolder, F.Cu at (174.0, 97.5)
- added Q1: MMBT2222A, Package_TO_SOT_SMD:SOT-23, F.Cu at (145.5, 81.4)
- added Q2: MMBT2222A, Package_TO_SOT_SMD:SOT-23, F.Cu at (152.0, 81.4)
- added Q3: MMBT2222A, Package_TO_SOT_SMD:SOT-23, F.Cu at (138.1, 81.3)
- added Q4: MMBT2222A, Package_TO_SOT_SMD:SOT-23, F.Cu at (144.8, 94.8)
- added R1: 1k, Resistor_SMD:R_1210_3225Metric_Pad1.30x2.65mm_HandSolder, F.Cu at (144.9, 103.0)
- added R2: 1k, Resistor_SMD:R_1210_3225Metric_Pad1.30x2.65mm_HandSolder, F.Cu at (146.5, 110.5)
- added R3: 4.7k, Resistor_SMD:R_1210_3225Metric_Pad1.30x2.65mm_HandSolder, F.Cu at (130.1, 78.0)
- added R4: 1k, Resistor_SMD:R_1210_3225Metric_Pad1.30x2.65mm_HandSolder, F.Cu at (145.5, 75.0)
- added R5: 1k, Resistor_SMD:R_1210_3225Metric_Pad1.30x2.65mm_HandSolder, F.Cu at (152.0, 75.0)
- added R6: 1k, Resistor_SMD:R_1210_3225Metric_Pad1.30x2.65mm_HandSolder, F.Cu at (139.0, 75.0)
- added R7: 1k, Resistor_SMD:R_1210_3225Metric_Pad1.30x2.65mm_HandSolder, F.Cu at (146.5, 89.0)
- added R8: 1k, Resistor_SMD:R_1210_3225Metric_Pad1.30x2.65mm_HandSolder, F.Cu at (181.4, 97.5)
- added U1: ~, Connector_PinHeader_2.54mm:PinHeader_1x08_P2.54mm_Vertical, F.Cu at (121.5, 86.0)
Routing:
- net Net-(Q2-C): track 0.00 -> 55.6 mm
- net Net-(Q1-C): track 0.00 -> 45.5 mm
- net Net-(Q4-C): track 0.00 -> 33.7 mm
- net Net-(U1-EL_SENS): track 0.00 -> 29.9 mm
- net Net-(Q3-C): track 0.00 -> 25.9 mm
- net Net-(A1-PadA0): track 0.00 -> 25.8 mm
- net Net-(A1-PadD8): track 0.00 -> 24.6 mm
- net Net-(U1-AZ_SENS): track 0.00 -> 22.6 mm
- net Net-(U1-PWR): track 0.00 -> 13.5 mm
- net Net-(A1-PadA1): track 0.00 -> 12.3 mm
- net Net-(A1-PadD6): track 0.00 -> 11.9 mm
- net Net-(A1-PadD9): track 0.00 -> 11.4 mm
- net Net-(A1-PadD10): track 0.00 -> 9.04 mm
- net Net-(A1-PadD7): track 0.00 -> 7.96 mm
- net Net-(Q4-B): track 0.00 -> 6.07 mm
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- added copper zone on B.Cu, net Earth
- added copper zone on F.Cu, net Earth
Other:
- board outline added: 86.6 x 53.9 mm
- rule pad_to_mask_clearance: 0 -> 0.09
- board text added: "YAESO G5500 Rotator Controller Shield for Arduino Mega"
