File: arduino-hat/arduino-hat.kicad_pcb (KiCad board)
At the start: 2 copper layers, 86.6 x 53.9 mm, 22 parts, among them Q1 MMBT2222A, Q2 MMBT2222A, Q3 MMBT2222A, Q4 MMBT2222A

Commit message: PCB design semi-finalized
Parts:
- removed C3: 10 uF, Capacitor_SMD:C_1210_3225Metric_Pad1.33x2.70mm_HandSolder
- removed R3: 4.7k, Resistor_SMD:R_1210_3225Metric_Pad1.30x2.65mm_HandSolder
- A1: footprint PCM_arduino-library:Arduino_Mega2560_R3_Shield -> PCM_arduino-library:Arduino_Mega2560_R3_Shield_revised
- C1, C2, C4, C5, C8, C9: footprint Capacitor_SMD:C_1210_3225Metric_Pad1.33x2.70mm_HandSolder -> Capacitor_SMD:C_0805_2012Metric_Pad1.18x1.45mm_HandSolder
- R1, R2, R4, R5, R6, R7, R8: footprint Resistor_SMD:R_1210_3225Metric_Pad1.30x2.65mm_HandSolder -> Resistor_SMD:R_0603_1608Metric_Pad0.98x0.95mm_HandSolder
- moved R2 0.67 mm to (146.7, 109.8)
Connections:
- A1 pad D10: Net-(A1-PadD10) -> unconnected-(A1-PadD10)
- U1 pad 1: Net-(U1-PWR) -> unconnected-(U1-PWR-Pad1)
Routing:
- net Net-(U1-PWR): track 13.5 -> 0.00 mm
- net Net-(A1-PadD10): track 9.04 -> 0.00 mm
- net Net-(Q4-B): track 6.07 -> 0.00 mm
- net Net-(A1-PadA1): track 12.3 -> 7.18 mm
- net Net-(A1-PadA0): track 25.8 -> 21.2 mm
- net Net-(A1-PadD9): track 11.4 -> 8.33 mm
- net Net-(U1-AZ_SENS): track 22.6 -> 23.5 mm
- net Net-(U1-EL_SENS): track 29.9 -> 30.5 mm
- net Net-(Q3-B): track 3.90 -> 4.54 mm
- net Net-(Q2-B): track 4.36 -> 4.99 mm
- net Net-(Q1-B): track 4.36 -> 4.99 mm
- net Net-(D1-A): track 4.41 -> 5.05 mm
- net Net-(A1-PadD42): track 4.39 -> 5.02 mm
- net Net-(A1-PadD8): track 24.6 -> 24.0 mm
