File: arduino-hat/arduino-hat.kicad_sch (KiCad schematic)
At the start: 20 parts, among them Q1 MMBT2222A, Q2 MMBT2222A, Q3 MMBT2222A, Q4 MMBT2222A

Commit message: finished?
Parts:
- D1: footprint LED_SMD:LED_1210_3225Metric_Pad1.42x2.65mm_HandSolder -> LED_SMD:LED_1206_3216Metric_Pad1.42x1.75mm_HandSolder
Changed lines of the file:
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@@
 			)
 		)
-		(property "Footprint" "LED_SMD:LED_1210_3225Metric_Pad1.42x2.65mm_HandSolder"
+		(property "Footprint" "LED_SMD:LED_1206_3216Metric_Pad1.42x1.75mm_HandSolder"
 			(at 165.1 148.59 0)
 			(effects
